File: placaPCB/planta_control.kicad_pcb (KiCad board)
At the start: 2 copper layers, 80 x 75 mm, 58 parts, among them J1 Conn_01x15_Pin, J2 USB_C_Receptacle, J3 Conn_01x15_Pin, J4 Conn_01x04_Pin, J5 Conn_01x06_Pin, J6 Conn_01x02_Pin, J7 Conn_01x02_Pin, Q1 MMBT3904, Q2 MMBT3904, SW1 SW_DIP_x01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

Commit message: .
.
Parts:
- removed C2, C3: 100uf, Capacitor_SMD:C_1206_3216Metric
- removed TP3: V_corriente_Q2, TestPoint:TestPoint_THTPad_1.0x1.0mm_Drill0.5mm
- removed TP4: V_corriente_Q1, TestPoint:TestPoint_THTPad_1.0x1.0mm_Drill0.5mm
- added G***: LOGO, logos:USCO2, F.Cu at (92.5, 97.5)
- R2, R3: value 1k -> 220
- moved SW1 1.00 mm to (34.3, 68.0)
- moved H4 0.50 mm to (102.0, 101.0)
- moved H3 0.46 mm to (28.0, 101.0)
Routing:
- net Net-(U2A-+): track 33.0 -> 25.8 mm
- net GND: track 432.2 -> 427.3 mm
- net Net-(U2B-+): track 34.7 -> 30.1 mm
- net vcc_esp: track 78.4 -> 79.4 mm
Other:
- board text added: "Desing: Cesar Muñoz"
- board text removed: "F1"
- board text removed: "F2"
