File: placaPCB/planta_control.kicad_sch (KiCad schematic)
At the start: 55 parts, among them J1 Conn_01x15_Pin, J2 USB_C_Receptacle, J3 Conn_01x15_Pin, J4 Conn_01x04_Pin, J5 Conn_01x06_Pin, J6 Conn_01x02_Pin, J7 Conn_01x02_Pin, Q1 MMBT3904, Q2 MMBT3904, SW1 SW_DIP_x01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

Commit message: .
.
Other:
- moved on the sheet: H1, H2, H3, H4, TP7, TP8, TP9
