File: planta_control.kicad_pcb (KiCad board)
At the start: 2 copper layers, 80 x 75 mm, 55 parts, among them J1 Conn_01x15_Pin, J2 USB_C_Receptacle, J3 Conn_01x15_Pin, J4 Conn_01x04_Pin, J5 Conn_01x06_Pin, J6 Conn_01x02_Pin, J7 Conn_01x02_Pin, Q1 MMBT3904, Q2 MMBT3904, SW1 SW_DIP_x01, T1 TIP31C, T2 TIP31C, U2 LM358, U3 DS18B20, U4 DS18B20, U5 DS18B20Z, U6 DS18B20Z

Commit message: .
.
Parts:
- removed the G*** at (92.5, 97.5)
- added G***: LOGO, Library:logoUsco, F.Cu at (92.5, 97.5)
- R12, R13, R2, R3, R6, R7: value 220 -> 150
Connections:
- J4 pad 2: vcc_esp -> +3.3V
- J5 pad 2: vcc_esp -> +3.3V
Routing:
- net vcc_esp: track 79.4 -> 13.5 mm
- net +3.3V: track 140.8 -> 203.4 mm, vias 4 -> 5
