File: _restore_backup_2026-09-26T16-56-07-640/planta_control.kicad_sch (KiCad schematic)
At the start: 55 parts, among them J1 Conn_01x15_Pin, J2 USB_C_Receptacle, J3 Conn_01x15_Pin, J4 Conn_01x04_Pin, J5 Conn_01x06_Pin, J6 Conn_01x02_Pin, J7 Conn_01x02_Pin, Q1 MMBT3904, Q2 MMBT3904, SW1 SW_DIP_x01, T1 TIP31C, T2 TIP31C, U1 ESp32, U2 LM358, U3 DS18B20, U4 DS18B20, U5 DS18B20Z, U6 DS18B20Z

Commit message: .
.
Changed lines of the file:
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@@
 	(wire
 		(pts
-			(xy 271.78 194.31) (xy 254 194.31)
+			(xy 265.43 194.31) (xy 254 194.31)
 		)
 		(stroke
@@
 	(wire
 		(pts
-			(xy 271.78 196.85) (xy 271.78 194.31)
+			(xy 265.43 195.58) (xy 265.43 194.31)
 		)
 		(stroke
@@
 	(wire
 		(pts
-			(xy 326.39 194.31) (xy 326.39 193.04)
+			(xy 331.47 194.31) (xy 331.47 193.04)
 		)
 		(stroke
@@
 	(wire
 		(pts
-			(xy 326.39 193.04) (xy 342.9 193.04)
+			(xy 331.47 193.04) (xy 342.9 193.04)
 		)
 		(stroke
@@
 	(symbol
 		(lib_id "power:GND")
-		(at 326.39 194.31 0)
+		(at 331.47 194.31 0)
 		(mirror y)
 		(unit 1)
@@
 		(fields_autoplaced yes)
 		(property "Reference" "#PWR01"
-			(at 326.39 200.66 0)
+			(at 331.47 200.66 0)
 			(hide yes)
 			(show_name no)
@@
 		)
 		(property "Value" "GND"
-			(at 326.39 199.39 0)
+			(at 331.47 199.39 0)
 			(show_name no)
 			(do_not_autoplace no)
@@
 		)
 		(property "Footprint" ""
-			(at 326.39 194.31 0)
+			(at 331.47 194.31 0)
 			(hide yes)
 			(show_name no)
@@
 		)
 		(property "Datasheet" ""
-			(at 326.39 194.31 0)
+			(at 331.47 194.31 0)
 			(hide yes)
 			(show_name no)
@@
 		)
 		(property "Description" "Power symbol creates a global label with name \"GND\" , ground"
-			(at 326.39 194.31 0)
+			(at 331.47 194.31 0)
 			(hide yes)
 			(show_name no)
@@
 	(symbol
 		(lib_id "power:GND")
-		(at 271.78 196.85 0)
+		(at 265.43 195.58 0)
 		(unit 1)
 		(body_style 1)
@@
 		(fields_autoplaced yes)
 		(property "Reference" "#PWR06"
-			(at 271.78 203.2 0)
+			(at 265.43 201.93 0)
 			(hide yes)
 			(show_name no)
@@
 		)
 		(property "Value" "GND"
-			(at 271.78 201.93 0)
+			(at 265.43 200.66 0)
 			(show_name no)
 			(do_not_autoplace no)
@@
 		)
 		(property "Footprint" ""
-			(at 271.78 196.85 0)
+			(at 265.43 195.58 0)
 			(hide yes)
 			(show_name no)
@@
 		)
 		(property "Datasheet" ""
-			(at 271.78 196.85 0)
+			(at 265.43 195.58 0)
 			(hide yes)
 			(show_name no)
@@
 		)
 		(property "Description" "Power symbol creates a global label with name \"GND\" , ground"
-			(at 271.78 196.85 0)
+			(at 265.43 195.58 0)
 			(hide yes)
 			(show_name no)
