File: .history/planta_control.kicad_pcb (KiCad board)
At the start: 2 copper layers, 80 x 75 mm, 58 parts, among them J1 Conn_01x15_Pin, J2 USB_C_Receptacle, J3 Conn_01x15_Pin, J4 Conn_01x04_Pin, J5 Conn_01x06_Pin, J6 Conn_01x02_Pin, J7 Conn_01x02_Pin, Q1 MMBT3904, Q2 MMBT3904, SW1 SW_DIP_x01, T1 TIP31C, T2 TIP31C, U2 LM358, U3 DS18B20, U4 DS18B20, U5 DS18B20Z, U6 DS18B20Z

Commit message: .
.
Parts:
- removed C2, C3: 100uf, Capacitor_SMD:C_1206_3216Metric
- removed TP3: V_corriente_Q2, TestPoint:TestPoint_THTPad_1.0x1.0mm_Drill0.5mm
- removed TP4: V_corriente_Q1, TestPoint:TestPoint_THTPad_1.0x1.0mm_Drill0.5mm
- added G***: LOGO, Library:logoUsco, F.Cu at (92.5, 97.5)
- R12, R13, R6, R7: value 220 -> 150
- R2, R3: value 1k -> 150
- moved SW1 1.00 mm to (34.3, 68.0)
Connections:
- J4 pad 2: vcc_esp -> +3.3V
- J5 pad 2: vcc_esp -> +3.3V
Routing:
- net vcc_esp: track 78.4 -> 13.5 mm
- net +3.3V: track 140.8 -> 203.4 mm, vias 4 -> 5
- net Net-(U2A-+): track 33.0 -> 25.8 mm
- net GND: track 432.2 -> 427.5 mm
- net Net-(U2B-+): track 34.7 -> 30.1 mm
Other:
- board text added: "Desing: Cesar Muñoz"
- board text removed: "F1"
- board text removed: "F2"

Commit message: .
.
Connections:
- J4 pad 2: +3.3V -> vcc_esp
- J5 pad 2: +3.3V -> vcc_esp
Routing:
- net +3.3V: track 203.4 -> 140.8 mm, vias 5 -> 4
- net vcc_esp: track 13.5 -> 75.7 mm
Changed lines of the file:
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@@
 			(layers "*.Cu" "*.Mask")
 			(remove_unused_layers no)
-			(net "+3.3V")
+			(net "vcc_esp")
 			(pinfunction "Pin_2_2")
 			(pintype "passive")
@@
 			)
 		)
+		(property "proyecto grado" ""
+			(at 0 0 0)
+			(unlocked yes)
+			(layer "F.Fab")
+			(hide yes)
+			(effects
+				(font
+					(size 1 1)
+					(thickness 0.25)
+				)
+			)
+		)
 		(sheetname "/")
 		(sheetfile "planta_control.kicad_sch")
@@
 			(layers "*.Cu" "*.Mask")
 			(remove_unused_layers no)
-			(net "+3.3V")
+			(net "vcc_esp")
 			(pinfunction "Pin_2_2")
 			(pintype "passive")
@@
 	)
 	(segment
-		(start 39.2234 87.5)
-		(end 39.2234 85.7766)
-		(width 0.8)
-		(layer "F.Cu")
-		(net "+3.3V")
-	)
-	(segment
-		(start 44.2205 80.7795)
-		(end 86.4503 80.7795)
-		(width 0.8)
-		(layer "F.Cu")
-		(net "+3.3V")
-	)
-	(segment
 		(start 69.5 48)
 		(end 68.3449 49.1551)
@@
 	)
 	(segment
-		(start 39.2234 85.7766)
-		(end 44.2205 80.7795)
-		(width 0.8)
-		(layer "F.Cu")
-		(net "+3.3V")
-	)
-	(segment
 		(start 78.5875 53.5875)
 		(end 80 53.5875)
@@
 	)
 	(via
-		(at 39.2234 87.5)
-		(size 1)
-		(drill 0.5)
-		(back_post_machining countersink
-			(angle 82)
-		)
-		(layers "F.Cu" "B.Cu")
-		(tenting
-			(front yes)
-			(back no)
-		)
-		(capping no)
-		(covering
-			(front no)
-			(back no)
-		)
-		(plugging
-			(front no)
-			(back no)
-		)
-		(filling no)
-		(net "+3.3V")
-	)
-	(via
 		(at 76.5 51.5)
 		(size 1)
@@
 	)
 	(segment
-		(start 96.5 84.46)
-		(end 92.8195 80.7795)
-		(width 0.8)
-		(layer "B.Cu")
-		(net "+3.3V")
-	)
-	(segment
 		(start 44.5 49.5)
 		(end 44.412596 49.5)
@@
 	)
 	(segment
-		(start 92.8195 80.7795)
-		(end 86.4503 80.7795)
-		(width 0.8)
-		(layer "B.Cu")
-		(net "+3.3V")
-	)
-	(segment
 		(start 44.412596 49.5)
 		(end 41.46 46.547404)
@@
 	)
 	(segment
+		(start 47.6176 80.7795)
+		(end 86.4503 80.7795)
+		(width 0.8)
+		(layer "F.Cu")
+		(net "vcc_esp")
+	)
+	(segment
 		(start 34.2675 68.9875)
 		(end 34.2675 67.9875)
@@
 	)
 	(segment
+		(start 39.2415 72.4034)
+		(end 47.6176 80.7795)
+		(width 0.8)
+		(layer "F.Cu")
+		(net "vcc_esp")
+	)
+	(segment
+		(start 96.5 84.46)
+		(end 92.8195 80.7795)
+		(width 0.8)
+		(layer "B.Cu")
+		(net "vcc_esp")
+	)
+	(segment
+		(start 92.8195 80.7795)
+		(end 86.4503 80.7795)
+		(width 0.8)
+		(layer "B.Cu")
+		(net "vcc_esp")
+	)
+	(segment
 		(start 49.5875 68.5875)
 		(end 51 70)
@@
 		)
 		(min_thickness 0.25)
-		(fill yes
+		(fill
 			(thermal_gap 0.5)
 			(thermal_bridge_width 0.5)

Commit message: .
.
Parts:
- U2: footprint Package_SO:SOIC-8_5.3x6.2mm_P1.27mm -> Package_SO:SOIC-8_3.9x4.9mm_P1.27mm
- moved G*** 0.25 mm to (92.5, 97.8)
Routing:
- net +3.3V: track 140.8 -> 143.1 mm
- net Net-(U2B--): track 15.6 -> 17.7 mm
- net GND: track 427.5 -> 428.6 mm
- net Net-(U2B-+): track 30.1 -> 31.1 mm
- net Net-(U2A--): track 17.9 -> 18.7 mm

Commit message: .
.
Connections:
- net AT1 renamed AT1/D26
- net AT2 renamed AT2/D25
- net MISO renamed MISO/D19
- net MOSI renamed MOSI/D23
- net Q1 renamed Q1/D13
- net Q2 renamed Q2/D12
- net SCK renamed SCK/D18
- net SCL renamed SCL/D22
- net SDA renamed SDA/D21
- net SS renamed SS/D15
- net T1 renamed T1/D14
- net T2 renamed T2/D27
- net Ven1 renamed Ven1/D33
- net Ven2 renamed Ven2/D32
- net corriente_Q1 renamed corriente_Q1/D35
- net corriente_Q2 renamed corriente_Q2/D34
- net vcc_esp renamed vcc_esp/vin
