File: .history/planta_control.kicad_sch (KiCad schematic)
At the start: 55 parts, among them J1 Conn_01x15_Pin, J2 USB_C_Receptacle, J3 Conn_01x15_Pin, J4 Conn_01x04_Pin, J5 Conn_01x06_Pin, J6 Conn_01x02_Pin, J7 Conn_01x02_Pin, Q1 MMBT3904, Q2 MMBT3904, SW1 SW_DIP_x01, T1 TIP31C, T2 TIP31C, U1 ESp32, U2 LM358, U3 DS18B20, U4 DS18B20, U5 DS18B20Z, U6 DS18B20Z

Commit message: .
.
Connections:
- net +3.3V: now also J4.2 (Pin_2), J5.2 (Pin_2)
- net vcc_esp: no longer J4.2 (Pin_2), J5.2 (Pin_2)
Changed lines of the file:
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@@
 	(wire
 		(pts
-			(xy 140.97 182.88) (xy 146.05 182.88)
+			(xy 140.97 182.88) (xy 149.86 182.88)
 		)
 		(stroke
@@
 	(wire
 		(pts
-			(xy 180.34 186.69) (xy 186.69 186.69)
+			(xy 180.34 186.69) (xy 189.23 186.69)
 		)
 		(stroke
@@
 		)
 	)
-	(global_label "vcc_esp"
-		(shape input)
-		(at 186.69 186.69 0)
-		(fields_autoplaced yes)
-		(effects
-			(font
-				(size 1.27 1.27)
-			)
-			(justify left)
-		)
-		(property "Intersheetrefs" "${INTERSHEET_REFS}"
-			(at 197.0533 186.69 0)
-			(hide yes)
-			(show_name no)
-			(do_not_autoplace no)
-			(effects
-				(font
-					(size 1.27 1.27)
-				)
-				(justify left)
-			)
-		)
-	)
 	(global_label "Q1"
 		(shape input)
@@
 		)
 	)
-	(global_label "vcc_esp"
-		(shape input)
-		(at 146.05 182.88 0)
-		(fields_autoplaced yes)
-		(effects
-			(font
-				(size 1.27 1.27)
-			)
-			(justify left)
-		)
-		(property "Intersheetrefs" "${INTERSHEET_REFS}"
-			(at 156.4133 182.88 0)
-			(hide yes)
-			(show_name no)
-			(do_not_autoplace no)
-			(effects
-				(font
-					(size 1.27 1.27)
-				)
-				(justify left)
-			)
-		)
-	)
 	(global_label "MOSI"
 		(shape input)
@@
 			)
 		)
+		(property "proyecto grado" ""
+			(at 175.26 97.79 0)
+			(show_name no)
+			(do_not_autoplace no)
+			(effects
+				(font
+					(size 1.27 1.27)
+				)
+			)
+		)
 		(pin "3"
 		)
@@
 	)
 	(symbol
+		(lib_id "power:+3.3V")
+		(at 149.86 182.88 270)
+		(unit 1)
+		(body_style 1)
+		(exclude_from_sim no)
+		(in_bom yes)
+		(on_board yes)
+		(in_pos_files yes)
+		(dnp no)
+		(fields_autoplaced yes)
+		(property "Reference" "#PWR035"
+			(at 146.05 182.88 0)
+			(hide yes)
+			(show_name no)
+			(do_not_autoplace no)
+			(effects
+				(font
+					(size 1.27 1.27)
+				)
+			)
+		)
+		(property "Value" "+3.3V"
+			(at 153.67 182.8799 90)
+			(show_name no)
+			(do_not_autoplace no)
+			(effects
+				(font
+					(size 1.27 1.27)
+				)
+				(justify left)
+			)
+		)
+		(property "Footprint" ""
+			(at 149.86 182.88 0)
+			(hide yes)
+			(show_name no)
+			(do_not_autoplace no)
+			(effects
+				(font
+					(size 1.27 1.27)
+				)
+			)
+		)
+		(property "Datasheet" ""
+			(at 149.86 182.88 0)
+			(hide yes)
+			(show_name no)
+			(do_not_autoplace no)
+			(effects
+				(font
+					(size 1.27 1.27)
+				)
+			)
+		)
+		(property "Description" "Power symbol creates a global label with name \"+3.3V\""
+			(at 149.86 182.88 0)
+			(hide yes)
+			(show_name no)
+			(do_not_autoplace no)
+			(effects
+				(font
+					(size 1.27 1.27)
+				)
+			)
+		)
+		(pin "1"
+		)
+		(instances
+			(project "planta_control"
+				(path "/0c8e7746-04af-4d75-a1b6-e1d457505b57"
+					(reference "#PWR035")
+					(unit 1)
+				)
+			)
+		)
+	)
+	(symbol
 		(lib_id "Transistor_BJT:MMBT3904")
 		(at 384.81 116.84 0)
@@
 					(unit 1)
 				)
+			)
+		)
+	)
+	(symbol
+		(lib_id "power:+3.3V")
+		(at 189.23 186.69 270)
+		(unit 1)
+		(body_style 1)
+		(exclude_from_sim no)
+		(in_bom yes)
+		(on_board yes)
+		(in_pos_files yes)
+		(dnp no)
+		(fields_autoplaced yes)
+		(property "Reference" "#PWR036"
+			(at 185.42 186.69 0)
+			(hide yes)
+			(show_name no)
+			(do_not_autoplace no)
+			(effects
+				(font
+					(size 1.27 1.27)
+				)
+			)
+		)
+		(property "Value" "+3.3V"
+			(at 193.04 186.6899 90)
+			(show_name no)
+			(do_not_autoplace no)
+			(effects
+				(font
+					(size 1.27 1.27)
+				)
+				(justify left)
+			)
+		)
+		(property "Footprint" ""
+			(at 189.23 186.69 0)
+			(hide yes)
+			(show_name no)
+			(do_not_autoplace no)
+			(effects
+				(font
+					(size 1.27 1.27)
+				)
+			)
+		)
+		(property "Datasheet" ""
+			(at 189.23 186.69 0)
+			(hide yes)
+			(show_name no)
+			(do_not_autoplace no)
+			(effects
+				(font
+					(size 1.27 1.27)
+				)
+			)
+		)
+		(property "Description" "Power symbol creates a global label with name \"+3.3V\""
+			(at 189.23 186.69 0)
+			(hide yes)
+			(show_name no)
+			(do_not_autoplace no)
+			(effects
+				(font
+					(size 1.27 1.27)
+				)
+			)
+		)
+		(pin "1"
+		)
+		(instances
+			(project "planta_control"
+				(path "/0c8e7746-04af-4d75-a1b6-e1d457505b57"
+					(reference "#PWR036")
+					(unit 1)
+				)

Commit message: .
.
Connections:
- net +3.3V: no longer J4.2 (Pin_2), J5.2 (Pin_2)
- net vcc_esp: now also J4.2 (Pin_2), J5.2 (Pin_2)
Changed lines of the file:
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@@
 	(wire
 		(pts
-			(xy 140.97 182.88) (xy 149.86 182.88)
+			(xy 140.97 182.88) (xy 146.05 182.88)
 		)
 		(stroke
@@
 	(wire
 		(pts
-			(xy 180.34 186.69) (xy 189.23 186.69)
+			(xy 180.34 186.69) (xy 186.69 186.69)
 		)
 		(stroke
@@
 		)
 	)
+	(global_label "vcc_esp"
+		(shape input)
+		(at 146.05 182.88 0)
+		(fields_autoplaced yes)
+		(effects
+			(font
+				(size 1.27 1.27)
+			)
+			(justify left)
+		)
+		(property "Intersheetrefs" "${INTERSHEET_REFS}"
+			(at 156.4133 182.88 0)
+			(hide yes)
+			(show_name no)
+			(do_not_autoplace no)
+			(effects
+				(font
+					(size 1.27 1.27)
+				)
+				(justify left)
+			)
+		)
+	)
 	(global_label "SS"
 		(shape input)
@@
 		)
 	)
+	(global_label "vcc_esp"
+		(shape input)
+		(at 186.69 186.69 0)
+		(fields_autoplaced yes)
+		(effects
+			(font
+				(size 1.27 1.27)
+			)
+			(justify left)
+		)
+		(property "Intersheetrefs" "${INTERSHEET_REFS}"
+			(at 197.0533 186.69 0)
+			(hide yes)
+			(show_name no)
+			(do_not_autoplace no)
+			(effects
+				(font
+					(size 1.27 1.27)
+				)
+				(justify left)
+			)
+		)
+	)
 	(global_label "T2"
 		(shape input)
@@
 	)
 	(symbol
-		(lib_id "power:+3.3V")
-		(at 149.86 182.88 270)
-		(unit 1)
-		(body_style 1)
-		(exclude_from_sim no)
-		(in_bom yes)
-		(on_board yes)
-		(in_pos_files yes)
-		(dnp no)
-		(fields_autoplaced yes)
-		(property "Reference" "#PWR035"
-			(at 146.05 182.88 0)
-			(hide yes)
-			(show_name no)
-			(do_not_autoplace no)
-			(effects
-				(font
-					(size 1.27 1.27)
-				)
-			)
-		)
-		(property "Value" "+3.3V"
-			(at 153.67 182.8799 90)
-			(show_name no)
-			(do_not_autoplace no)
-			(effects
-				(font
-					(size 1.27 1.27)
-				)
-				(justify left)
-			)
-		)
-		(property "Footprint" ""
-			(at 149.86 182.88 0)
-			(hide yes)
-			(show_name no)
-			(do_not_autoplace no)
-			(effects
-				(font
-					(size 1.27 1.27)
-				)
-			)
-		)
-		(property "Datasheet" ""
-			(at 149.86 182.88 0)
-			(hide yes)
-			(show_name no)
-			(do_not_autoplace no)
-			(effects
-				(font
-					(size 1.27 1.27)
-				)
-			)
-		)
-		(property "Description" "Power symbol creates a global label with name \"+3.3V\""
-			(at 149.86 182.88 0)
-			(hide yes)
-			(show_name no)
-			(do_not_autoplace no)
-			(effects
-				(font
-					(size 1.27 1.27)
-				)
-			)
-		)
-		(pin "1"
-		)
-		(instances
-			(project "planta_control"
-				(path "/0c8e7746-04af-4d75-a1b6-e1d457505b57"
-					(reference "#PWR035")
-					(unit 1)
-				)
-			)
-		)
-	)
-	(symbol
 		(lib_id "Transistor_BJT:MMBT3904")
 		(at 384.81 116.84 0)
@@
 					(unit 1)
 				)
-			)
-		)
-	)
-	(symbol
-		(lib_id "power:+3.3V")
-		(at 189.23 186.69 270)
-		(unit 1)
-		(body_style 1)
-		(exclude_from_sim no)
-		(in_bom yes)
-		(on_board yes)
-		(in_pos_files yes)
-		(dnp no)
-		(fields_autoplaced yes)
-		(property "Reference" "#PWR036"
-			(at 185.42 186.69 0)
-			(hide yes)
-			(show_name no)
-			(do_not_autoplace no)
-			(effects
-				(font
-					(size 1.27 1.27)
-				)
-			)
-		)
-		(property "Value" "+3.3V"
-			(at 193.04 186.6899 90)
-			(show_name no)
-			(do_not_autoplace no)
-			(effects
-				(font
-					(size 1.27 1.27)
-				)
-				(justify left)
-			)
-		)
-		(property "Footprint" ""
-			(at 189.23 186.69 0)
-			(hide yes)
-			(show_name no)
-			(do_not_autoplace no)
-			(effects
-				(font
-					(size 1.27 1.27)
-				)
-			)
-		)
-		(property "Datasheet" ""
-			(at 189.23 186.69 0)
-			(hide yes)
-			(show_name no)
-			(do_not_autoplace no)
-			(effects
-				(font
-					(size 1.27 1.27)
-				)
-			)
-		)
-		(property "Description" "Power symbol creates a global label with name \"+3.3V\""
-			(at 189.23 186.69 0)
-			(hide yes)
-			(show_name no)
-			(do_not_autoplace no)
-			(effects
-				(font
-					(size 1.27 1.27)
-				)
-			)
-		)
-		(pin "1"
-		)
-		(instances
-			(project "planta_control"
-				(path "/0c8e7746-04af-4d75-a1b6-e1d457505b57"
-					(reference "#PWR036")
-					(unit 1)
-				)

Commit message: .
.
Parts:
- U2: footprint Package_SO:SOIC-8_5.3x6.2mm_P1.27mm -> Package_SO:SOIC-8_3.9x4.9mm_P1.27mm
Changed lines of the file:
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@@
 	(wire
 		(pts
-			(xy 265.43 194.31) (xy 254 194.31)
+			(xy 271.78 194.31) (xy 254 194.31)
 		)
 		(stroke
@@
 	(wire
 		(pts
-			(xy 265.43 195.58) (xy 265.43 194.31)
+			(xy 271.78 196.85) (xy 271.78 194.31)
 		)
 		(stroke
@@
 	(wire
 		(pts
-			(xy 331.47 194.31) (xy 331.47 193.04)
+			(xy 326.39 194.31) (xy 326.39 193.04)
 		)
 		(stroke
@@
 	(wire
 		(pts
-			(xy 331.47 193.04) (xy 342.9 193.04)
+			(xy 326.39 193.04) (xy 342.9 193.04)
 		)
 		(stroke
@@
 	(symbol
 		(lib_id "power:GND")
-		(at 331.47 194.31 0)
+		(at 326.39 194.31 0)
 		(mirror y)
 		(unit 1)
@@
 		(fields_autoplaced yes)
 		(property "Reference" "#PWR01"
-			(at 331.47 200.66 0)
+			(at 326.39 200.66 0)
 			(hide yes)
 			(show_name no)
@@
 		)
 		(property "Value" "GND"
-			(at 331.47 199.39 0)
+			(at 326.39 199.39 0)
 			(show_name no)
 			(do_not_autoplace no)
@@
 		)
 		(property "Footprint" ""
-			(at 331.47 194.31 0)
+			(at 326.39 194.31 0)
 			(hide yes)
 			(show_name no)
@@
 		)
 		(property "Datasheet" ""
-			(at 331.47 194.31 0)
+			(at 326.39 194.31 0)
 			(hide yes)
 			(show_name no)
@@
 		)
 		(property "Description" "Power symbol creates a global label with name \"GND\" , ground"
-			(at 331.47 194.31 0)
+			(at 326.39 194.31 0)
 			(hide yes)
 			(show_name no)
@@
 			)
 		)
-		(property "Footprint" "Package_SO:SOIC-8_5.3x6.2mm_P1.27mm"
+		(property "Footprint" "Package_SO:SOIC-8_3.9x4.9mm_P1.27mm"
 			(at 201.93 114.3 0)
 			(hide yes)
@@
 			)
 		)
-		(property "Footprint" "Package_SO:SOIC-8_5.3x6.2mm_P1.27mm"
+		(property "Footprint" "Package_SO:SOIC-8_3.9x4.9mm_P1.27mm"
 			(at 201.93 54.61 0)
 			(hide yes)
@@
 	(symbol
 		(lib_id "power:GND")
-		(at 265.43 195.58 0)
+		(at 271.78 196.85 0)
 		(unit 1)
 		(body_style 1)
@@
 		(fields_autoplaced yes)
 		(property "Reference" "#PWR06"
-			(at 265.43 201.93 0)
+			(at 271.78 203.2 0)
 			(hide yes)
 			(show_name no)
@@
 		)
 		(property "Value" "GND"
-			(at 265.43 200.66 0)
+			(at 271.78 201.93 0)
 			(show_name no)
 			(do_not_autoplace no)
@@
 		)
 		(property "Footprint" ""
-			(at 265.43 195.58 0)
+			(at 271.78 196.85 0)
 			(hide yes)
 			(show_name no)
@@
 		)
 		(property "Datasheet" ""
-			(at 265.43 195.58 0)
+			(at 271.78 196.85 0)
 			(hide yes)
 			(show_name no)
@@
 		)
 		(property "Description" "Power symbol creates a global label with name \"GND\" , ground"
-			(at 265.43 195.58 0)
+			(at 271.78 196.85 0)
 			(hide yes)
 			(show_name no)
@@
 			)
 		)
-		(property "Footprint" "Package_SO:SOIC-8_5.3x6.2mm_P1.27mm"
+		(property "Footprint" "Package_SO:SOIC-8_3.9x4.9mm_P1.27mm"
 			(at 210.82 29.21 0)
 			(hide yes)

Commit message: .
.
Parts:
- removed U1: ESp32, Library_new:ESP32_Node_MCU_30_Pines_2.5mm, symbol creados:Esp32_NodeMCU
Connections:
- net AT1 renamed AT1/D26
- net AT2 renamed AT2/D25
- net MISO renamed MISO/D19
- net MOSI renamed MOSI/D23
- net Q1 renamed Q1/D13
- net Q2 renamed Q2/D12
- net SCK renamed SCK/D18
- net SCL renamed SCL/D22
- net SDA renamed SDA/D21
- net SS renamed SS/D15
- net T1 renamed T1/D14
- net T2 renamed T2/D27
- net Ven1 renamed Ven1/D33
- net Ven2 renamed Ven2/D32
- net corriente_Q1 renamed corriente_Q1/D35
- net corriente_Q2 renamed corriente_Q2/D34
- net vcc_esp renamed vcc_esp/vin
- no-connect marks 36 -> 26
Other:
- moved on the sheet: C1, D1, D2, H1, H2, H3, H4, J1, J2, J3, R1, R10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
